File: DymBOX_AVR.kicad_sch (KiCad schematic)
At the start: 26 parts, among them J2 Conn_01x03_Pin, J3 Conn_01x02_Pin, J4 Conn_01x03_Pin, J5 Conn_02x05_Odd_Even, Q3 BS170, Q4 BS170, SW1 RotaryEncoder_Switch, U1 ATmega8A-P, U2 CA56-12EWA, U3 L7805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

Commit message: pcb
Parts:
- added Q1: BC327, Package_TO_SOT_THT:TO-92L_HandSolder, symbol Transistor_BJT:BC327
- added Q2, Q5: BC327, Package_TO_SOT_THT:TO-92_HandSolder, symbol Transistor_BJT:BC327
- added R10, R11, R12: R, Resistor_THT:R_Axial_DIN0204_L3.6mm_D1.6mm_P5.08mm_Horizontal, symbol Device:R
Connections:
- net +5V: now also Q1.3 (E), Q2.3 (E), Q5.3 (E)
- net SEG_C: now also U1.26 (PC3); no longer U1.23 (PC0)
- net SEG_D: now also U1.24 (PC1); no longer U1.26 (PC3)
- net SEG_E: now also U1.23 (PC0); no longer U1.27 (PC4)
- net SEG_G: now also U1.27 (PC4); no longer U1.24 (PC1)
- net DIG_0: now reaches U1.2 (PD0)
- net DIG_0: now also R10.1
- net DIG_1: now reaches U1.3 (PD1)
- net DIG_1: now also R11.1
- net DIG_2: now reaches U1.4 (PD2)
- net DIG_2: now also R12.1
- net at U2.6 (CA4): now also Q1.1 (C)
- net at U2.8 (CA3): now also Q2.1 (C)
- net at U2.9 (CA2): now also Q5.1 (C)
- new net: Q1.2 (B), R10.2
- new net: Q2.2 (B), R11.2
- new net: Q5.2 (B), R12.2
- no-connect marks 3 -> 4
Other:
- moved on the sheet: Q3, Q4, SW1

Commit message: pcb_f
Parts:
- removed J2: Conn_01x03_Pin, Connector_Phoenix_MC:PhoenixContact_MCV_1,5_3-G-3.5_1x03_P3.50mm_Vertical, symbol Connector:Conn_01x03_Pin
- added J1: Conn_01x04_Pin, Connector_Phoenix_MC:PhoenixContact_MCV_1,5_4-G-3.5_1x04_P3.50mm_Vertical, symbol Connector:Conn_01x04_Pin
- added R13: 4k7, Resistor_THT:R_Axial_DIN0204_L3.6mm_D1.6mm_P5.08mm_Horizontal, symbol Device:R
- added R14, R15: 330, Resistor_THT:R_Axial_DIN0204_L3.6mm_D1.6mm_P5.08mm_Horizontal, symbol Device:R
- added R16, R17: 10k, Resistor_THT:R_Axial_DIN0204_L3.6mm_D1.6mm_P5.08mm_Horizontal, symbol Device:R
- C3, C4, C5, C6: footprint Capacitor_THT:C_Disc_D10.0mm_W2.5mm_P5.00mm -> Capacitor_THT:C_Disc_D5.0mm_W2.5mm_P5.00mm
- J4: value Conn_01x03_Pin -> DS18B20
- R1: footprint Resistor_THT:R_Axial_DIN0207_L6.3mm_D2.5mm_P10.16mm_Horizontal -> Resistor_THT:R_Axial_DIN0204_L3.6mm_D1.6mm_P5.08mm_Horizontal
- SW1: footprint (none) -> Rotary_Encoder:RotaryEncoder_Alps_EC12E-Switch_Vertical_H20mm_CircularMountingHoles
- U3: footprint Package_TO_SOT_THT:TO-220F-3_Horizontal_TabDown -> Package_TO_SOT_THT:TO-220-3_Horizontal_TabDown
- Y1: footprint Crystal:Crystal_SMD_HC49-SD_HandSoldering -> Crystal:Crystal_HC49-U_Vertical
Connections:
- net +12V: now also J1.2 (Pin_2), J1.4 (Pin_4)
- net +5V: now also J4.3 (Pin_3), R13.2
- net GND: now also J4.1 (Pin_1), J5.3 (Pin_3), J5.8 (Pin_8), Q3.3 (S), Q4.3 (S), SW1.C, SW1.S2, R16.1, R17.1; no longer J4.3 (Pin_3)
- net CLK: now reaches SW1.A
- net CLK: now also U1.5 (PD3)
- net DT: now reaches SW1.B
- net DT: now also U1.6 (PD4)
- net BTN: now reaches SW1.S1
- net BTN: now also U1.11 (PD5)
- net at U1.15 (PB1): now also R14.1
- net at U1.16 (PB2): now also R15.1
- net MOSI: now reaches U1.17 (PB3)
- net MOSI: now also J5.1 (Pin_1)
- net MISO: now reaches U1.18 (PB4)
- net MISO: now also J5.9 (Pin_9)
- net SCK: now reaches U1.19 (PB5)
- net SCK: now also J5.7 (Pin_7)
- net at U1.28 (PC5): now also J4.2 (Pin_2), R13.1
- net at Q3.1 (D): now also J1.3 (Pin_3)
- net at Q3.2 (G): now also R14.2, R16.2
- net at Q4.1 (D): now also J1.1 (Pin_1)
- net at Q4.2 (G): now also R15.2, R17.2
- no-connect marks 4 -> 3
Other:
- moved on the sheet: C1, C2, C3, J3, J4, Q1, Q2, Q3, Q4, Q5, R10, R11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

Commit message: pcb_transfo
Parts:
- removed J1: Conn_01x04_Pin, Connector_Phoenix_MC:PhoenixContact_MCV_1,5_4-G-3.5_1x04_P3.50mm_Vertical, symbol Connector:Conn_01x04_Pin
- removed J3: Conn_01x02_Pin, Connector_Phoenix_MC:PhoenixContact_MCV_1,5_2-G-3.5_1x02_P3.50mm_Vertical, symbol Connector:Conn_01x02_Pin
- added D1, D2: 1N4148, Diode_THT:D_DO-35_SOD27_P7.62mm_Horizontal, symbol Diode:1N4148
- added D3: D_Bridge_+-AA, Diode_THT:Diode_Bridge_DIP-4_W5.08mm_P2.54mm, symbol Device:D_Bridge_+-AA
- added F1: Fuse, Fuse:Fuseholder_Clip-5x20mm_Littelfuse_111_Inline_P20.00x5.00mm_D1.05mm_Horizontal, symbol Device:Fuse
- added J6, J7, J8, J9: Conn_01x01_Pin, 2pkstartup:TRM2_62409-1_TEC, symbol 2pkstartup:FST
- added K1: RT314A24, Relay_THT:Relay_SPDT_Schrack-RT1-16A-FormC_RM5mm, symbol Relay:RT314A24
- added TR1: TEZ6.0-D-1, Transformer_THT:Transformer_Breve_TEZ-38x45, symbol Transformer:TEZ6.0-D-1
- C1, C2: footprint Capacitor_THT:CP_Radial_D10.0mm_P7.50mm -> Capacitor_THT:CP_Radial_D13.0mm_P5.00mm
- C5: value C_Small -> Q1
- J4: footprint Connector_Phoenix_MC:PhoenixContact_MCV_1,5_3-G-3.5_1x03_P3.50mm_Vertical -> Connector_Wire:SolderWire-0.127sqmm_1x03_P3.7mm_D0.48mm_OD1mm
- Q1: footprint Package_TO_SOT_THT:TO-92L_HandSolder -> Package_TO_SOT_THT:TO-92_HandSolder
- Q3, Q4: footprint Package_TO_SOT_THT:TO-92_Inline -> Package_TO_SOT_THT:TO-92_HandSolder
- R1: value R -> 10k
- R10, R11, R12: value R -> 1k
- Y1: value Crystal -> 16MHz
Connections:
- net +12V: now also D1.1 (K), D2.1 (K), F1.1, K1.A1
- net BTN: now also U1.2 (PD0); no longer U1.11 (PD5)
- net DIG_0: now also U1.3 (PD1); no longer U1.2 (PD0)
- net DIG_1: now also U1.4 (PD2); no longer U1.3 (PD1)
- net DIG_2: now also U1.12 (PD6); no longer U1.4 (PD2)
- net GND: now also D3.2 (-)
- net SEG_B: now also U1.11 (PD5); no longer U1.12 (PD6)
- net at Q3.1 (D): now also D1.2 (A)
- net at Q4.1 (D): now also D2.2 (A), K1.A2
- new net: D3.1 (+), F1.2
- new net: J8.1 (Pin_1), K1.11
- new net: J6.1 (Pin_1), TR1.5
- new net: D3.3, TR1.9
- new net: D3.4, TR1.7
- new net: J7.1 (Pin_1), TR1.1
- new net: J9.1 (Pin_1), K1.14
Other:
- moved on the sheet: C1, C2, C3, C4, C5, C6, J4, J5, Q1, Q2, Q3, Q4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
